File: Schematics & pcb layout/KiCad/arduino-fanatec-pcb.sch (KiCad schematic (older format))
At the start: 16 parts, among them J1 SPI Connector 01x08_Female, J2 TM1637 4 digit Display connec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, J3 Breakout Connector 02x18_Odd_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, U1 Simple_Chinese_Logic_level_sh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

Commit message: wip
Connections:
- net GND: no longer J1.3 (Pin_3), J1.5 (Pin_5), U1.12 (GND-L)
- new net: J1.3 (Pin_3), J1.5 (Pin_5), U1.12 (GND-L)
Changed lines of the file:
@@
 	7000 4600 7150 4600
 Connection ~ 4750 2200
-Wire Wire Line
-	3900 5350 4100 5350
-Connection ~ 3900 5350
-Connection ~ 4100 5350
 Text Label 6550 4550 0    50   ~ 0
 Dpad
