File: Pro Mini V2 3.3V/eagle pcb files/board.sch (EAGLE design)
At the start: 4 parts, among them X1 B8B-PH-KL, X2 87758-0216

Commit message: #9 Update readme and PCB files
- add wheelbase damage warning
- add note to uncomment lines
- remove connection of 5V to RAW (including diode)
Parts:
- removed D1: 1N4004, adafruit:1N4004
Connections:
- removed net RAW: D1.C, U$7.RAW
- net 4_5V: no longer D1.A
Changed lines of the file:
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@@
 <part name="U$7" library="Arduino-clone" deviceset="PRO-MINI_5BOT" device="" override_package3d_urn="urn:adsk.eagle:package:23456791/2" override_package_urn="urn:adsk.eagle:footprint:23456792/1"/>
 <part name="U$8" library="microbuilder" deviceset="GND" device=""/>
-<part name="D1" library="adafruit" library_urn="urn:adsk.eagle:library:420" deviceset="1N4004" device="" package3d_urn="urn:adsk.eagle:package:6240344/1" override_package3d_urn="urn:adsk.eagle:package:23456826/2" override_package_urn="urn:adsk.eagle:footprint:6239679/1"/>
 <part name="U$9" library="microbuilder" deviceset="GND" device=""/>
 <part name="U$10" library="microbuilder" deviceset="GND" device=""/>
@@
 <instance part="U$8" gate="G$1" x="-12.7" y="127" smashed="yes">
 <attribute name="VALUE" x="-14.224" y="124.46" size="1.27" layer="96"/>
-</instance>
-<instance part="D1" gate="1" x="-22.86" y="142.24" smashed="yes">
-<attribute name="NAME" x="-20.32" y="142.7226" size="1.778" layer="95"/>
-<attribute name="VALUE" x="-20.32" y="139.9286" size="1.778" layer="96"/>
 </instance>
 <instance part="U$9" gate="G$1" x="12.7" y="149.86" smashed="yes" rot="MR0">
@@
 <segment>
 <label x="-33.02" y="142.24" size="1.778" layer="95"/>
-<pinref part="D1" gate="1" pin="A"/>
 <pinref part="X1" gate="G$1" pin="8"/>
-<wire x1="-25.4" y1="142.24" x2="-43.18" y2="142.24" width="0.1524" layer="91"/>
 <pinref part="X2" gate="-2" pin="S"/>
 <wire x1="-38.1" y1="114.3" x2="-43.18" y2="114.3" width="0.1524" layer="91"/>
 <wire x1="-43.18" y1="114.3" x2="-43.18" y2="142.24" width="0.1524" layer="91"/>
-<junction x="-43.18" y="142.24"/>
 </segment>
 </net>
-<net name="RAW" class="0">
-<segment>
-<pinref part="D1" gate="1" pin="C"/>
-<wire x1="-20.32" y1="142.24" x2="-17.78" y2="142.24" width="0.1524" layer="91"/>
-<wire x1="-17.78" y1="142.24" x2="-17.78" y2="185.42" width="0.1524" layer="91"/>
-<wire x1="-17.78" y1="185.42" x2="60.96" y2="185.42" width="0.1524" layer="91"/>
-<wire x1="60.96" y1="185.42" x2="60.96" y2="165.1" width="0.1524" layer="91"/>
-<pinref part="U$7" gate="G$1" pin="RAW"/>
-<wire x1="60.96" y1="165.1" x2="58.42" y2="165.1" width="0.1524" layer="91"/>
-</segment>
-</net>
